Commit message: add real robot

File: pybullet_gym/pybullet_ur5/assets/ur_description/ur10_joint_limited_robot.urdf (robot description, URDF)
Before this commit: robot ur5, 11 links, 10 joints
Links:
- link base_link: geometry collision mesh filename=package://ur_description/meshes/ur10/collision/base.stl; visual mesh filename=package://ur_description/meshes/ur10/visual/base.dae
- link forearm_link: mass 2.275 -> 3.87; geometry collision mesh filename=package://ur_description/meshes/ur10/collision/forearm.stl; visual mesh filename=package://ur_description/meshes/ur10/visual/forearm.dae
- link shoulder_link: mass 3.7 -> 7.778; geometry collision mesh filename=package://ur_description/meshes/ur10/collision/shoulder.stl; visual mesh filename=package://ur_description/meshes/ur10/visual/shoulder.dae
- link upper_arm_link: mass 8.393 -> 12.93; geometry collision mesh filename=package://ur_description/meshes/ur10/collision/upperarm.stl; visual mesh filename=package://ur_description/meshes/ur10/visual/upperarm.dae
- link wrist_1_link: mass 1.219 -> 1.96; geometry collision mesh filename=package://ur_description/meshes/ur10/collision/wrist1.stl; visual mesh filename=package://ur_description/meshes/ur10/visual/wrist1.dae
- link wrist_2_link: mass 1.219 -> 1.96; geometry collision mesh filename=package://ur_description/meshes/ur10/collision/wrist2.stl; visual mesh filename=package://ur_description/meshes/ur10/visual/wrist2.dae
- link wrist_3_link: mass 0.1879 -> 0.202; geometry collision mesh filename=package://ur_description/meshes/ur10/collision/wrist3.stl; visual mesh filename=package://ur_description/meshes/ur10/visual/wrist3.dae
Joints:
- joint base_link-base_fixed_joint: origin xyz=0 0 0 rpy=0 0 -3.141592653589793 -> xyz=0 0 0 rpy=0 0 -3.14159265359
- joint ee_fixed_joint: origin xyz=0.0 0.0823 0.0 rpy=0.0 0.0 1.5707963267948966 -> xyz=0.0 0.0922 0.0 rpy=0.0 0.0 1.57079632679
- joint elbow_joint: limit lower=-3.141592653589793 upper=3.141592653589793 effort=150.0 velocity=3.15 -> lower=-3.14159265359 upper=3.14159265359 effort=150.0 velocity=3.15; origin xyz=0.0 -0.1197 0.425 rpy=0.0 0.0 0.0 -> xyz=0.0 -0.1719 0.612 rpy=0.0 0.0 0.0
- joint shoulder_lift_joint: limit lower=-3.14 upper=3.14 effort=150.0 velocity=3.15 -> lower=-3.14159265359 upper=3.14159265359 effort=330.0 velocity=2.16; origin xyz=0.0 0.13585 0.0 rpy=0.0 1.5707963267948966 0.0 -> xyz=0.0 0.220941 0.0 rpy=0.0 1.57079632679 0.0
- joint shoulder_pan_joint: limit lower=-3.14 upper=3.14 effort=150.0 velocity=3.15 -> lower=-3.14159265359 upper=3.14159265359 effort=330.0 velocity=2.16; origin xyz=0.0 0.0 0.089159 rpy=0.0 0.0 -3.1415926 -> xyz=0.0 0.0 0.1273 rpy=0.0 0.0 0.0
- joint wrist_1_joint: limit lower=-3.14 upper=3.14 effort=28.0 velocity=3.2 -> lower=-3.14159265359 upper=3.14159265359 effort=54.0 velocity=3.2; origin xyz=0.0 0.0 0.39225 rpy=0.0 1.5707963267948966 0.0 -> xyz=0.0 0.0 0.5723 rpy=0.0 1.57079632679 0.0
- joint wrist_2_joint: limit lower=-3.14 upper=3.14 effort=28.0 velocity=3.2 -> lower=-3.14159265359 upper=3.14159265359 effort=54.0 velocity=3.2; origin xyz=0.0 0.093 0.0 rpy=0.0 0.0 0.0 -> xyz=0.0 0.1149 0.0 rpy=0.0 0.0 0.0
- joint wrist_3_joint: limit lower=-3.14 upper=3.14 effort=28.0 velocity=3.2 -> lower=-3.14159265359 upper=3.14159265359 effort=54.0 velocity=3.2; origin xyz=0.0 0.0 0.09465 rpy=0.0 0.0 0.0 -> xyz=0.0 0.0 0.1157 rpy=0.0 0.0 0.0
- joint wrist_3_link-tool0_fixed_joint: origin xyz=0 0.0823 0 rpy=-1.5707963267948966 0 0 -> xyz=0 0.0922 0 rpy=-1.57079632679 0 0

File: pybullet_gym/pybullet_ur5/assets/ur_description/ur10_robot.urdf (robot description, URDF)
Before this commit: robot ur5, 11 links, 10 joints
Links:
- link base_link: geometry collision mesh filename=package://ur_description/meshes/ur10/collision/base.stl; visual mesh filename=package://ur_description/meshes/ur10/visual/base.dae
- link forearm_link: mass 2.275 -> 3.87; geometry collision mesh filename=package://ur_description/meshes/ur10/collision/forearm.stl; visual mesh filename=package://ur_description/meshes/ur10/visual/forearm.dae
- link shoulder_link: mass 3.7 -> 7.778; geometry collision mesh filename=package://ur_description/meshes/ur10/collision/shoulder.stl; visual mesh filename=package://ur_description/meshes/ur10/visual/shoulder.dae
- link upper_arm_link: mass 8.393 -> 12.93; geometry collision mesh filename=package://ur_description/meshes/ur10/collision/upperarm.stl; visual mesh filename=package://ur_description/meshes/ur10/visual/upperarm.dae
- link wrist_1_link: mass 1.219 -> 1.96; geometry collision mesh filename=package://ur_description/meshes/ur10/collision/wrist1.stl; visual mesh filename=package://ur_description/meshes/ur10/visual/wrist1.dae
- link wrist_2_link: mass 1.219 -> 1.96; geometry collision mesh filename=package://ur_description/meshes/ur10/collision/wrist2.stl; visual mesh filename=package://ur_description/meshes/ur10/visual/wrist2.dae
- link wrist_3_link: mass 0.1879 -> 0.202; geometry collision mesh filename=package://ur_description/meshes/ur10/collision/wrist3.stl; visual mesh filename=package://ur_description/meshes/ur10/visual/wrist3.dae
Joints:
- joint base_link-base_fixed_joint: origin xyz=0 0 0 rpy=0 0 -3.141592653589793 -> xyz=0 0 0 rpy=0 0 -3.14159265359
- joint ee_fixed_joint: origin xyz=0.0 0.0823 0.0 rpy=0.0 0.0 1.5707963267948966 -> xyz=0.0 0.0922 0.0 rpy=0.0 0.0 1.57079632679
- joint elbow_joint: limit lower=-3.141592653589793 upper=3.141592653589793 effort=150.0 velocity=3.15 -> lower=-3.14159265359 upper=3.14159265359 effort=150.0 velocity=3.15; origin xyz=0.0 -0.1197 0.425 rpy=0.0 0.0 0.0 -> xyz=0.0 -0.1719 0.612 rpy=0.0 0.0 0.0
- joint shoulder_lift_joint: limit lower=-3.14 upper=3.14 effort=150.0 velocity=3.15 -> lower=-6.28318530718 upper=6.28318530718 effort=330.0 velocity=2.16; origin xyz=0.0 0.13585 0.0 rpy=0.0 1.5707963267948966 0.0 -> xyz=0.0 0.220941 0.0 rpy=0.0 1.57079632679 0.0
- joint shoulder_pan_joint: limit lower=-3.14 upper=3.14 effort=150.0 velocity=3.15 -> lower=-6.28318530718 upper=6.28318530718 effort=330.0 velocity=2.16; origin xyz=0.0 0.0 0.089159 rpy=0.0 0.0 -3.1415926 -> xyz=0.0 0.0 0.1273 rpy=0.0 0.0 0.0
- joint wrist_1_joint: limit lower=-3.14 upper=3.14 effort=28.0 velocity=3.2 -> lower=-6.28318530718 upper=6.28318530718 effort=54.0 velocity=3.2; origin xyz=0.0 0.0 0.39225 rpy=0.0 1.5707963267948966 0.0 -> xyz=0.0 0.0 0.5723 rpy=0.0 1.57079632679 0.0
- joint wrist_2_joint: limit lower=-3.14 upper=3.14 effort=28.0 velocity=3.2 -> lower=-6.28318530718 upper=6.28318530718 effort=54.0 velocity=3.2; origin xyz=0.0 0.093 0.0 rpy=0.0 0.0 0.0 -> xyz=0.0 0.1149 0.0 rpy=0.0 0.0 0.0
- joint wrist_3_joint: limit lower=-3.14 upper=3.14 effort=28.0 velocity=3.2 -> lower=-6.28318530718 upper=6.28318530718 effort=54.0 velocity=3.2; origin xyz=0.0 0.0 0.09465 rpy=0.0 0.0 0.0 -> xyz=0.0 0.0 0.1157 rpy=0.0 0.0 0.0
- joint wrist_3_link-tool0_fixed_joint: origin xyz=0 0.0823 0 rpy=-1.5707963267948966 0 0 -> xyz=0 0.0922 0 rpy=-1.57079632679 0 0
