Commit message: old ur5

File: pybullet_gym/pybullet_ur5/assets/ur_description/ur5.urdf (robot description, URDF)
Before this commit: robot ur5, 11 links, 10 joints
Joints:
- joint shoulder_pan_joint: limit lower=-3.14 upper=3.14 effort=150.0 velocity=3.15 -> lower=-3.14 upper=3.5 effort=150.0 velocity=3.15

Commit message: 3.31

File: pybullet_gym/pybullet_ur5/assets/ur_description/ur5.urdf (robot description, URDF)
Before this commit: robot ur5, 11 links, 10 joints
Joints:
- joint shoulder_pan_joint: limit lower=-3.14 upper=3.5 effort=150.0 velocity=3.15 -> lower=-3.14 upper=3.8 effort=150.0 velocity=3.15
