Commit message: add both arms optimization

File: pybullet_gym/pybullet_ur5/assets/kinect_human/upper_body_left.urdf (robot description, URDF)
Before this commit: robot upper_body, 31 links, 30 joints
Links:
- removed link ElbowRight
- removed link ShoulderRight
- removed link head_link
- removed link right_elbow
- removed link right_elbow_psi_link
- removed link right_elbow_theta_link
- removed link right_hand
- removed link right_lower_arm
- removed link right_shoulder_link
- removed link right_shoulder_theta_link
- removed link right_spine_phi_link
- removed link right_spine_theta_link
- removed link right_spine_to_shoulde_link
- removed link right_upper_arm
- link SpineLink: geometry visual cylinder length=0.4 radius=0.05
Joints:
- removed joint LShoulderSY
- removed joint LShoulderSZ
- removed joint RElbowX
- removed joint RElbowY
- removed joint RElbowZ
- removed joint RShoulderSY
- removed joint RShoulderSZ
- removed joint RShoulderX
- removed joint RShoulderY
- removed joint RShoulderZ
- removed joint fix_head_joint
- removed joint left_shoulder_fixed
- removed joint right_elbow_fixed3
- removed joint right_fix_elbow_joint
- removed joint right_hand_fixed
- removed joint right_should_fixed
- removed joint right_shoulder_fixed
- added joint ShoulderSY: type continuous, parent shoulder_spine_link, child left_spine_theta_link, axis 0 1 0
- added joint ShoulderSZ: type continuous, parent left_spine_theta_link, child left_spine_phi_link, axis 0 0 1
- added joint Shoulder_fixed: type fixed, parent left_spine_phi_link, child left_spine_to_shoulde_link, origin xyz=0.08 0 0 rpy=0 1.57 0
