Commit message: add optimization

File: pybullet_gym/pybullet_ur5/assets/kinect_human/upper_body bc.urdf (robot description, URDF)
Before this commit: robot upper_body, 13 links, 12 joints
Links:
- removed link ElbowLeft
- removed link ShoulderLeft
- removed link SpineBase
- removed link left_shoulder_link
- removed link shoulder_spine_link
- removed link world
- added link body_link
- added link head_link; visual sphere radius=0.10
- added link left_elbow3
- added link left_shoulder; visual sphere radius=0.05
- added link left_shoulder3
- added link left_shoulder_psi_link
- added link right_shoulder; visual sphere radius=0.05
- added link right_shoulder3
- added link right_shoulder_psi_link
- added link right_shoulder_theta_link
- added link right_upper_arm; visual cylinder length=0.25 radius=0.03
- link left_elbow: geometry visual sphere radius=0.05
- link left_lower_arm: geometry visual cylinder length=0.25 radius=0.02
- link left_upper_arm: geometry visual cylinder length=0.25 radius=0.03
Joints:
- removed joint base_spine_joint
- removed joint left_should_fixed
- removed joint shoulder_spine_joint
- added joint RShoulderX: type continuous, parent right_shoulder, child right_shoulder_psi_link, axis 1 0 0
- added joint RShoulderY: type continuous, parent right_shoulder_psi_link, child right_shoulder_theta_link, axis 0 1 0
- added joint RShoulderZ: type continuous, parent right_shoulder_theta_link, child right_shoulder3, axis 0 0 1
- added joint fix_head_joint: type fixed, parent body_link, child head_link, origin xyz=0.0 0 0.32 rpy=0.0 0.0 0.0
- added joint left_fix_shoulder_joint: type fixed, parent body_link, child left_shoulder, origin xyz=0.25 -0.05 0.25 rpy=1.57 0 0.0
- added joint left_should_fixed3: type fixed, parent left_shoulder3, child left_upper_arm, origin xyz=0.125 0 0.0 rpy=0 1.57 0
- added joint right_fix_shoulder_joint: type fixed, parent body_link, child right_shoulder, origin xyz=-0.25 -0.05 0.25 rpy=1.57 -1.57 0.0
- added joint right_should_fixed3: type fixed, parent right_shoulder3, child right_upper_arm, origin xyz=-0.125 0 0.0 rpy=0 1.57 0
- joint LElbowZ: child ElbowLeft -> left_elbow3
- joint LShoulderX: child left_shoulder_link -> left_shoulder_psi_link; origin xyz=0.18 0 0.0 rpy=0 0 -1.57 -> (none); parent shoulder_spine_link -> left_shoulder
- joint LShoulderY: parent left_shoulder_link -> left_shoulder_psi_link
- joint LShoulderZ: child ShoulderLeft -> left_shoulder3
- joint left_elbow_fixed3: origin xyz=0 0.14 0 rpy=1.57 0 0.0 -> xyz=0 0.125 0 rpy=1.57 0 0.0; parent ElbowLeft -> left_elbow3
- joint left_fix_elbow_joint: origin xyz=0 0.0 0.14 rpy=1.57 0 3.14 -> xyz=0 0.0 0.125 rpy=1.57 0 3.14
- joint left_hand_fixed: origin xyz=0 0 -0.14 rpy=0 0 0.0 -> xyz=0 0 -0.125 rpy=-1.57 0 0.0

Commit message: update environment

File: pybullet_gym/pybullet_ur5/assets/kinect_human/upper_body bc.urdf (robot description, URDF)
Before this commit: robot upper_body, 18 links, 17 joints
Links:
- added link human_base
- link body_link: geometry visual mesh filename=spine.STL
Joints:
- added joint base_body_joint: type fixed, parent human_base, child body_link, origin xyz=0.0 0 0 rpy=0.0 0.0 0.0

File: pybullet_gym/pybullet_ur5/assets/kinect_human/upper_body.urdf (robot description, URDF)
Before this commit: robot upper_body, 29 links, 28 joints
Links:
- link SpineLink: geometry visual mesh filename=spine.STL scale=0.8 1 1
