Commit message: update urdf

File: pybullet_gym/pybullet_ur5/assets/kinect_human/upper_body.urdf (robot description, URDF)
Before this commit: robot upper_body, 13 links, 12 joints
Links:
- added link SpineLink; visual cylinder length=0.4 radius=0.05
- added link left_spine_theta_link
- added link left_spine_to_shoulde_link; visual cylinder length=0.16 radius=0.02
- link SpineBase: geometry visual sphere radius=0.05
Joints:
- added joint ShoulderSY: type continuous, parent shoulder_spine_link, child left_spine_theta_link, axis 0 1 0
- added joint ShoulderSZ: type continuous, parent left_spine_theta_link, child left_spine_to_shoulde_link, origin xyz=0.08 0 0 rpy=0 1.57 0, axis 0 1 0
- added joint spine_joint: type fixed, parent SpineBase, child SpineLink, origin xyz=0 0.2 0 rpy=1.57 0 0.0
- joint LShoulderX: origin xyz=0.18 0 0.0 rpy=0 0 -1.57 -> xyz=0 0 0.08 rpy=1.57 0 -1.57; parent shoulder_spine_link -> left_spine_to_shoulde_link
- joint shoulder_spine_joint: origin xyz=0 0.45 0 rpy=0 0 0.0 -> xyz=0 0 -0.2 rpy=-1.57 0 0.0; parent SpineBase -> SpineLink

Commit message: left arm

File: pybullet_gym/pybullet_ur5/assets/kinect_human/upper_body.urdf (robot description, URDF)
Before this commit: robot upper_body, 16 links, 15 joints
Links:
- added link left_spine_phi_link
- link left_upper_arm: geometry visual cylinder length=0.24 radius=0.03
Joints:
- added joint Shoulder_fixed: type fixed, parent left_spine_phi_link, child left_spine_to_shoulde_link, origin xyz=0.08 0 0 rpy=0 1.57 0
- joint ShoulderSZ: axis 0 1 0 -> 0 0 1; child left_spine_to_shoulde_link -> left_spine_phi_link; origin xyz=0.08 0 0 rpy=0 1.57 0 -> (none)
- joint left_elbow_fixed3: origin xyz=0 0.14 0 rpy=1.57 0 0.0 -> xyz=0 0.12 0 rpy=1.57 0 0.0
- joint left_fix_elbow_joint: origin xyz=0 0.0 0.14 rpy=1.57 0 3.14 -> xyz=0 0.0 0.12 rpy=1.57 0 3.14
- joint left_hand_fixed: origin xyz=0 0 -0.14 rpy=0 0 0.0 -> xyz=0 0 -0.12 rpy=0 0 0.0
- joint left_should_fixed: origin xyz=0.14 0 0.0 rpy=0 1.57 0 -> xyz=0.12 0 0.0 rpy=0 1.57 0

Commit message: add both arms

File: pybullet_gym/pybullet_ur5/assets/kinect_human/upper_body.urdf (robot description, URDF)
Before this commit: robot upper_body, 31 links, 30 joints
Links:
- link left_upper_arm: geometry visual cylinder length=0.22 radius=0.03
- link right_upper_arm: geometry visual cylinder length=0.22 radius=0.03
Joints:
- joint left_elbow_fixed3: origin xyz=0 0.12 0 rpy=1.57 0 0.0 -> xyz=0 0.11 0 rpy=1.57 0 0.0
- joint left_fix_elbow_joint: origin xyz=0 0.0 0.12 rpy=1.57 0 3.14 -> xyz=0 0.0 0.11 rpy=1.57 0 3.14
- joint left_hand_fixed: origin xyz=0 0 -0.12 rpy=0 0 0.0 -> xyz=0 0 -0.11 rpy=0 0 0.0
- joint left_should_fixed: origin xyz=0.12 0 0.0 rpy=0 1.57 0 -> xyz=0.11 0 0.0 rpy=0 1.57 0
- joint right_elbow_fixed3: origin xyz=0 0.12 0 rpy=1.57 0 0.0 -> xyz=0 0.11 0 rpy=1.57 0 0.0
- joint right_fix_elbow_joint: origin xyz=0 0.0 -0.12 rpy=-1.57 0 0 -> xyz=0 0.0 -0.11 rpy=-1.57 0 0
- joint right_hand_fixed: origin xyz=0 0 -0.12 rpy=0 0 0.0 -> xyz=0 0 -0.11 rpy=0 0 0.0
- joint right_should_fixed: origin xyz=-0.12 0 0.0 rpy=0 1.57 0 -> xyz=-0.11 0 0.0 rpy=0 1.57 0

Commit message: add human optimization

File: pybullet_gym/pybullet_ur5/assets/kinect_human/upper_body.urdf (robot description, URDF)
Before this commit: robot upper_body, 31 links, 30 joints
Links:
- removed link left_hand
- removed link right_hand
- added link WristLeft; visual sphere radius=0.05
- added link WristRight; visual sphere radius=0.05
Joints:
- joint left_hand_fixed: child left_hand -> WristLeft
- joint right_hand_fixed: child right_hand -> WristRight

Commit message: test

File: pybullet_gym/pybullet_ur5/assets/kinect_human/upper_body.urdf (robot description, URDF)
Before this commit: robot upper_body, 31 links, 30 joints
Links:
- link SpineBase: geometry collision sphere radius=0.05; visual sphere radius=0.05
- link SpineLink: geometry collision cylinder length=0.4 radius=0.08; visual cylinder length=0.4 radius=0.08
- link WristLeft: geometry collision sphere radius=0.05; visual sphere radius=0.05
- link WristRight: geometry collision sphere radius=0.05; visual sphere radius=0.05
- link head_link: geometry collision sphere radius=0.07; visual sphere radius=0.07
- link left_elbow: geometry collision sphere radius=0.02; visual sphere radius=0.02
- link left_lower_arm: geometry collision cylinder length=0.28 radius=0.02; visual cylinder length=0.28 radius=0.02
- link left_shoulder_link: geometry collision sphere radius=0.02; visual sphere radius=0.02
- link left_spine_to_shoulde_link: geometry collision cylinder length=0.16 radius=0.02; visual cylinder length=0.16 radius=0.02
- link left_upper_arm: geometry collision cylinder length=0.22 radius=0.03; visual cylinder length=0.22 radius=0.03
- link right_elbow: geometry collision sphere radius=0.02; visual sphere radius=0.02
- link right_lower_arm: geometry collision cylinder length=0.28 radius=0.02; visual cylinder length=0.28 radius=0.02
- link right_shoulder_link: geometry collision sphere radius=0.02; visual sphere radius=0.02
- link right_spine_to_shoulde_link: geometry collision cylinder length=0.16 radius=0.02; visual cylinder length=0.16 radius=0.02
- link right_upper_arm: geometry collision cylinder length=0.22 radius=0.03; visual cylinder length=0.22 radius=0.03
- link shoulder_spine_link: geometry collision sphere radius=0.05; visual sphere radius=0.05

Commit message: adjust weight

File: pybullet_gym/pybullet_ur5/assets/kinect_human/upper_body.urdf (robot description, URDF)
Before this commit: robot upper_body, 31 links, 30 joints
Links:
- removed link left_elbow_theta_link
- removed link right_elbow_theta_link
- link SpineLink: geometry collision cylinder length=0.4 radius=0.08; visual box size=0.1 0.05 0.4
- link left_lower_arm: geometry collision cylinder length=0.28 radius=0.04; visual cylinder length=0.28 radius=0.04
- link left_upper_arm: geometry collision cylinder length=0.22 radius=0.05; visual cylinder length=0.22 radius=0.05
- link right_lower_arm: geometry collision cylinder length=0.28 radius=0.04; visual cylinder length=0.28 radius=0.04
- link right_upper_arm: geometry collision cylinder length=0.22 radius=0.05; visual cylinder length=0.22 radius=0.05
Joints:
- removed joint LElbowY
- removed joint RElbowY
- joint LElbowZ: parent left_elbow_theta_link -> left_elbow_psi_link
- joint RElbowZ: parent right_elbow_theta_link -> right_elbow_psi_link

Commit message: add rnn policy

File: pybullet_gym/pybullet_ur5/assets/kinect_human/upper_body.urdf (robot description, URDF)
Before this commit: robot upper_body, 29 links, 28 joints
Links:
- link left_spine_to_shoulde_link: geometry collision cylinder length=0.16 radius=0.03; visual cylinder length=0.16 radius=0.03
- link right_spine_to_shoulde_link: geometry collision cylinder length=0.16 radius=0.03; visual cylinder length=0.16 radius=0.03
