Commit message: add demonstration

File: pybullet_gym/pybullet_ur5/assets/scenes_data/cylinder/cylinder.urdf (robot description, URDF)
Before this commit: robot targetball, 1 links, 0 joints
Links:
- link boxLink: geometry collision cylinder length=0.25 radius=0.06; visual cylinder length=0.25 radius=0.06

Commit message: add arm urdf

File: pybullet_gym/pybullet_ur5/assets/scenes_data/cylinder/cylinder.urdf (robot description, URDF)
Before this commit: robot cylinder, 1 links, 0 joints
Links:
- removed link boxLink
- added link elbow_link, mass .0; collision sphere radius=0.06; visual sphere radius=0.06
- added link forearm_link, mass .0; collision cylinder length=0.25 radius=0.06; visual cylinder length=0.25 radius=0.06
- added link hand_link, mass .0; collision sphere radius=0.07; visual sphere radius=0.07
Joints:
- added joint elbow_fixed_joint: type fixed, parent forearm_link, child elbow_link, origin xyz=0.0 0.0 -0.15 rpy=0.0 0.0 0.0
- added joint hand_fixed_joint: type fixed, parent forearm_link, child hand_link, origin xyz=0.0 0.0 0.15 rpy=0.0 0.0 0.0

Commit message: working version 1

File: pybullet_gym/pybullet_ur5/assets/scenes_data/cylinder/cylinder.urdf (robot description, URDF)
Before this commit: robot cylinder, 3 links, 2 joints
Links:
- link elbow_link: geometry collision sphere radius=0.05; visual sphere radius=0.05
- link forearm_link: geometry collision cylinder length=0.22 radius=0.04; visual cylinder length=0.22 radius=0.04
- link hand_link: geometry collision sphere radius=0.06; visual sphere radius=0.06

Commit message: working version

File: pybullet_gym/pybullet_ur5/assets/scenes_data/cylinder/cylinder.urdf (robot description, URDF)
Before this commit: robot cylinder, 3 links, 2 joints
Links:
- link elbow_link: geometry collision sphere radius=0.06; visual sphere radius=0.06
- link forearm_link: geometry collision cylinder length=0.22 radius=0.055; visual cylinder length=0.22 radius=0.055
- link hand_link: geometry collision sphere radius=0.07; visual sphere radius=0.07

Commit message: ddpg version

File: pybullet_gym/pybullet_ur5/assets/scenes_data/cylinder/cylinder.urdf (robot description, URDF)
Before this commit: robot cylinder, 3 links, 2 joints
Links:
- link elbow_link: geometry collision sphere radius=0.05; visual sphere radius=0.05
- link forearm_link: geometry collision cylinder length=0.22 radius=0.05; visual cylinder length=0.22 radius=0.05
- link hand_link: geometry collision sphere radius=0.06; visual sphere radius=0.06

Commit message: 1. add user recording 2. add batch q and real time collision avoidance

File: pybullet_gym/pybullet_ur5/assets/scenes_data/cylinder/cylinder.urdf (robot description, URDF)
Before this commit: robot cylinder, 3 links, 2 joints
Links:
- link elbow_link: geometry collision sphere radius=0.04; visual sphere radius=0.04
- link forearm_link: geometry collision cylinder length=0.22 radius=0.04; visual cylinder length=0.22 radius=0.04
- link hand_link: geometry collision sphere radius=0.05; visual sphere radius=0.05

Commit message: test for ly

File: pybullet_gym/pybullet_ur5/assets/scenes_data/cylinder/cylinder.urdf (robot description, URDF)
Before this commit: robot cylinder, 3 links, 2 joints
Links:
- link elbow_link: geometry collision sphere radius=0.00; visual sphere radius=0.00
- link forearm_link: geometry collision cylinder length=0.12 radius=0.00; visual cylinder length=0.12 radius=0.00
- link hand_link: geometry collision sphere radius=0.00; visual sphere radius=0.00

Commit message: fix pyik problem

File: pybullet_gym/pybullet_ur5/assets/scenes_data/cylinder/cylinder.urdf (robot description, URDF)
Before this commit: robot cylinder, 3 links, 2 joints
Links:
- link elbow_link: geometry collision sphere radius=0.02; visual sphere radius=0.02
- link forearm_link: geometry collision cylinder length=0.22 radius=0.02; visual cylinder length=0.22 radius=0.02

Commit message: fix bugs

File: pybullet_gym/pybullet_ur5/assets/scenes_data/cylinder/cylinder.urdf (robot description, URDF)
Before this commit: robot cylinder, 3 links, 2 joints
Links:
- link elbow_link: geometry collision sphere radius=0.03; visual sphere radius=0.03
- link forearm_link: geometry collision cylinder length=0.22 radius=0.02; visual cylinder length=0.22 radius=0.02
- link hand_link: geometry collision sphere radius=0.03; visual sphere radius=0.03
